File: Hardware/Prototype_2/PCB/PCB.kicad_pcb (KiCad board)
At the start: 2 copper layers, 66 x 45.7 mm, 7 parts, among them J1 Bluetooth Interface, J2 Powerboost, J3 GSR Header, J4 PPG Header, U1 ARDUINO_MICRO_SHIELD

Commit message: PCB Final Version, Added Gerber Files
Parts:
- removed J4: PPG Header, Connector_PinHeader_2.00mm:PinHeader_1x06_P2.00mm_Vertical
- added D1: LED, LED_THT:LED_D3.0mm_Horizontal_O1.27mm_Z6.0mm, F.Cu at (142.2, 82.1)
- added J5: Screw_Terminal_01x02, TerminalBlock:TerminalBlock_Altech_AK300-2_P5.00mm, F.Cu at (150.9, 50.3)
- added J6: Screw_Terminal_01x02, TerminalBlock:TerminalBlock_Altech_AK300-2_P5.00mm, F.Cu at (139.1, 50.4)
- added J7: Screw_Terminal_01x02, TerminalBlock:TerminalBlock_Altech_AK300-2_P5.00mm, F.Cu at (142.0, 65.5)
- added R3: 1K, Resistor_THT:R_Axial_DIN0204_L3.6mm_D1.6mm_P7.62mm_Horizontal, F.Cu at (146.3, 70.2)
- added S1: EG1218, digikey-footprints:Switch_Slide_11.6x4mm_EG1218, F.Cu at (137.2, 74.9)
- J2: footprint Connector_PinHeader_2.00mm:PinHeader_1x08_P2.00mm_Vertical -> Connector_PinSocket_2.54mm:PinSocket_1x08_P2.54mm_Vertical
- R1: value 3.3K -> 2K
- R2: value 1.1K -> 1K
- moved J1 66.4 mm to (196.6, 51.3), turned to 180 degrees
- moved R2 13.1 mm to (141.6, 70.2), turned to -90 degrees
- moved R1 12.1 mm to (144.0, 70.2), turned to -90 degrees
- moved J2 6.53 mm to (188.7, 65.9)
- moved J3 4.04 mm to (157.5, 65.5), turned to 180 degrees
Connections:
- J1 pad 2: Net-(J1-Pad2) -> +5V
- J1 pad 3: Net-(J1-Pad3) -> GND
- J1 pad 4: GND -> Net-(J1-Pin_4)
- J1 pad 5: +5V -> Net-(J1-Pin_5)
- R1 pad 2: Net-(J1-Pad2) -> Net-(J1-Pin_5)
- R2 pad 2: Net-(J1-Pad2) -> Net-(J1-Pin_5)
- U1 pad A1: Net-(J1-Pad3) -> Net-(J1-Pin_4)
Routing:
- net Net-(J1-Pin_5): track 0.00 -> 75.6 mm, vias 0 -> 2
- net Net-(J6-Pin_1): track 0.00 -> 69.7 mm, vias 0 -> 2
- net Net-(J5-Pin_1): track 0.00 -> 59.0 mm, vias 0 -> 1
- net /PowerBoost_EN: track 0.00 -> 58.8 mm, vias 0 -> 3
- net Net-(J5-Pin_2): track 0.00 -> 56.2 mm, vias 0 -> 1
- net Net-(J6-Pin_2): track 0.00 -> 55.7 mm, vias 0 -> 2
- net Net-(J1-Pad3): track 53.9 -> 0.00 mm, vias 2 -> 0
- net Net-(J1-Pin_4): track 0.00 -> 26.3 mm
- net +5V: track 0.00 -> 20.1 mm, vias 0 -> 1
- net unconnected-(U1-RESET-PadRST): track 0.00 -> 15.3 mm
- net Net-(J1-Pad2): track 13.7 -> 0.00 mm
- net Net-(J3-Pin_4): track 29.8 -> 43.3 mm
- net GND: track 0.00 -> 8.69 mm, vias 0 -> 1
- net Net-(D1-A): track 0.00 -> 6.82 mm
- net Net-(J2-Pin_3): track 0.00 -> 6.53 mm
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Other:
- board size 66 x 45.7 mm -> 64.4 x 45.7 mm
