File: Hardware/Prototype_2/PCB/PCB.kicad_sch (KiCad schematic)
At the start: 7 parts, among them J1 Bluetooth Interface, J2 Powerboost, J3 GSR Header, J4 PPG Header, U1 ARDUINO_MICRO_SHIELD

Commit message: PCB Final Version, Added Gerber Files
Parts:
- removed J4: PPG Header, Connector_PinHeader_2.00mm:PinHeader_1x06_P2.00mm_Vertical, symbol Connector:Screw_Terminal_01x06
- added D1: LED, LED_THT:LED_D3.0mm_Horizontal_O1.27mm_Z6.0mm, symbol Device:LED
- added J5, J6, J7: Screw_Terminal_01x02, TerminalBlock:TerminalBlock_Altech_AK300-2_P5.00mm, symbol Connector:Screw_Terminal_01x02
- added R3: 1K, Resistor_THT:R_Axial_DIN0204_L3.6mm_D1.6mm_P7.62mm_Horizontal, symbol Device:R
- added S1: EG1218, digikey-footprints:Switch_Slide_11.6x4mm_EG1218, symbol dk_Slide-Switches:EG1218
- J2: footprint Connector_PinHeader_2.00mm:PinHeader_1x08_P2.00mm_Vertical -> Connector_PinSocket_2.54mm:PinSocket_1x08_P2.54mm_Vertical
- R1: value 3.3K -> 2K
- R2: value 1.1K -> 1K
Connections:
- net +3V3: now also J7.1 (Pin_1)
- net +5V: now also J1.2 (Pin_2), D1.1 (K); no longer J1.5 (Pin_5)
- net GND: now also J1.3 (Pin_3), J7.2 (Pin_2), R3.1, S1.2; no longer J1.4 (Pin_4)
- net PowerBoost_EN: now also S1.1
- net at U1.5 (5(PWM)): now also J5.1 (Pin_1)
- net at U1.4 (4/A6): now also J5.2 (Pin_2)
- net at U1.3 (3(PWM)/SCL): now also J6.1 (Pin_1)
- net at U1.2 (2/SDA): now also J6.2 (Pin_2)
- net at R1.2, R2.2: now also J1.5 (Pin_5); no longer J1.2 (Pin_2)
- net at U1.A1: now also J1.4 (Pin_4); no longer J1.3 (Pin_3)
- new net: D1.2 (A), R3.2
- no-connect marks 6 -> 26
Other:
- moved on the sheet: J1
